File: chervil8or_PCB/_autosave-chervil8or.sch (KiCad schematic (older format))
At the start: 58 parts, among them J1 TRRS_MJ-4PP-9, J2 TRRS_MJ-4PP-9, J3 TRRS_MJ-4PP-9, J4 TRRS_MJ-4PP-9, SW1 SW_PUSH, SW10 SW_PUSH, SW11 SW_PUSH, SW12 SW_PUSH, SW13 SW_PUSH, SW14 SW_PUSH, SW15 SW_PUSH, SW16 SW_PUSH, SW17 SW_PUSH, SW18 Rotary_Encoder_Switch, SW2 SW_PUSH, SW3 SW_PUSH, SW4 SW_PUSH, SW5 SW_PUSH, SW6 SW_PUSH, SW7 SW_PUSH, SW8 SW_PUSH, SW9 Rotary_Encoder_Switch, U1 ProMicro, U2 ProMicro

Commit message: fix
Parts:
- added H1, H10, H11, H12, H13, H14, H15, H16, H17, H18, H19, H2, H20, H21, H22, H23, H24, H25, H26, H27, H28, H29, H3, H30, H31, H32, H4, H5, H6, H7, H8, H9: MountingHole, kbd_Hole:m2_Screw_Hole, symbol Mechanical:MountingHole
- renumbered D2 to D1, D20 to D10, D21 to D11, D23 to D12, D26 to D13, D28 to D14, D29 to D15, D31 to D16, D4 to D2, D5 to D3, D7 to D4, D10 to D5, D12 to D6, D13 to D7, D15 to D8, D18 to D9
