File: chervil8or_PCB/chervil8or.kicad_pcb (KiCad board)
At the start: 2 copper layers, 190.2 x 166.1 mm, 134 parts, among them J1 TRRS_MJ-4PP-9, J2 TRRS_MJ-4PP-9, J3 TRRS_MJ-4PP-9, J4 TRRS_MJ-4PP-9, SW1 SW_PUSH, SW10 SW_PUSH, SW11 SW_PUSH, SW12 SW_PUSH, SW13 SW_PUSH, SW14 SW_PUSH, SW15 SW_PUSH, SW16 SW_PUSH, SW17 SW_PUSH, SW18 Rotary_Encoder_Switch, SW2 SW_PUSH, SW3 SW_PUSH, SW4 SW_PUSH, SW5 SW_PUSH, SW6 SW_PUSH, SW7 SW_PUSH, SW8 SW_PUSH, SW9 Rotary_Encoder_Switch, U1 ProMicro, U2 ProMicro

Commit message: fix
Parts:
- removed the D1 at (31.0, 11.9)
- removed the D11 at (31.0, 59.5)
- removed the D12 at (33.3, 59.5)
- removed the D14 at (50.0, 57.1)
- removed the D16 at (50.0, 61.9)
- removed D17, D19, D22, D24, D25, D27, D30, D32: D, kbd_Parts:Diode_TH_SMD
- removed the D3 at (31.0, 21.4)
- removed the D8 at (33.3, 40.5)
- removed the D9 at (31.0, 50.0)
- removed Ref** (x23): Val**, kbd_Hole:Mouse_Bite_Hole
- removed the Ref1 at (-9.23, -8.33)
- added Ref13: Val13, kbd_Hole:Mouse_Bite_Hole, F.Cu at (66.7, 69.9)
- added Ref14: Val14, kbd_Hole:Mouse_Bite_Hole, F.Cu at (66.7, 73.5)
- added Ref15: Val15, kbd_Hole:Mouse_Bite_Hole, F.Cu at (124.7, 69.9)
- added Ref16: Val16, kbd_Hole:Mouse_Bite_Hole, F.Cu at (124.7, 73.5)
- added Ref17: Val17, kbd_Hole:Mouse_Bite_Hole, F.Cu at (140.2, 69.9)
- added Ref18: Val18, kbd_Hole:Mouse_Bite_Hole, F.Cu at (140.2, 73.5)
- added Ref19: Val19, kbd_Hole:Mouse_Bite_Hole, F.Cu at (172.6, 69.9)
- added Ref20: Val20, kbd_Hole:Mouse_Bite_Hole, F.Cu at (172.6, 73.5)
- added Ref23: Val23, kbd_Hole:Mouse_Bite_Hole, F.Cu at (130.7, 79.5)
- added Ref24: Val24, kbd_Hole:Mouse_Bite_Hole, F.Cu at (134.2, 79.5)
- added Ref28: Val28, kbd_Hole:Mouse_Bite_Hole, F.Cu at (130.7, 149.4)
- added Ref29: Val29, kbd_Hole:Mouse_Bite_Hole, F.Cu at (134.2, 149.4)
- added Ref8: Val8, kbd_Hole:Mouse_Bite_Hole, F.Cu at (134.2, 64.0)
- added Rf1: Val1, kbd_Hole:m2_Screw_Hole, F.Cu at (-9.23, -8.33)
- added Rf10: Val10, kbd_Hole:m2_Screw_Hole, F.Cu at (64.3, 66.4)
- added Rf11: Val11, kbd_Hole:m2_Screw_Hole, F.Cu at (89.9, 66.4)
- added Rf12: Val12, kbd_Hole:m2_Screw_Hole, F.Cu at (127.1, 66.4)
- added Rf2: Val2, kbd_Hole:m2_Screw_Hole, F.Cu at (28.0, -8.33)
- added Rf3: Val3, kbd_Hole:m2_Screw_Hole, F.Cu at (39.0, 35.4)
- added Rf4: Val4, kbd_Hole:m2_Screw_Hole, F.Cu at (-9.23, 66.4)
- added Rf5: Val5, kbd_Hole:m2_Screw_Hole, F.Cu at (28.0, 66.4)
- added Rf6: Val6, kbd_Hole:m2_Screw_Hole, F.Cu at (53.6, 66.4)
- added Rf7: Val7, kbd_Hole:m2_Screw_Hole, F.Cu at (89.9, -8.33)
- added Rf9: Val9, kbd_Hole:m2_Screw_Hole, F.Cu at (79.2, 36.0)
- R16: renamed from Ref5; value Val5 -> Val16
- Ref1: renamed from Ref**; value Val** -> Val1
- Ref10, Ref11, Ref12, Ref2, Ref3, Ref4, Ref5, Ref6, Ref7, Ref9: footprint kbd_Hole:m2_Screw_Hole -> kbd_Hole:Mouse_Bite_Hole
- Ref21: renamed from Ref**; value Val** -> Val21
- Ref22: renamed from Ref**; value Val** -> Val22
- Ref26: renamed from Ref**; value Val** -> Val26
- Ref27: renamed from Ref**; value Val** -> Val27
- Rf13: renamed from Ref1; value Val1 -> Val13
- Rf14: renamed from Ref2; value Val2 -> Val14
- Rf15: renamed from Ref4; value Val4 -> Val15
- Rf17: renamed from Ref1; value Val1 -> Val17
- Rf18: renamed from Ref2; value Val2 -> Val18
- Rf19: renamed from Ref3; value Val3 -> Val19
- Rf20: renamed from Ref4; value Val4 -> Val20
- Rf21: renamed from Ref5; value Val5 -> Val21
- Rf22: renamed from Ref6; value Val6 -> Val22
- Rf23: renamed from Ref7; value Val7 -> Val23
- Rf24: renamed from Ref8; value Val8 -> Val24
- Rf25: renamed from Ref9; value Val9 -> Val25
- Rf26: renamed from Ref10; value Val10 -> Val26
- Rf27: renamed from Ref11; value Val11 -> Val27
- Rf28: renamed from Ref12; value Val12 -> Val28
- Rf29: renamed from Ref7; value Val7 -> Val29
- Rf30: renamed from Ref8; value Val8 -> Val30
- Rf31: renamed from Ref11; value Val11 -> Val31
- Rf32: renamed from Ref12; value Val12 -> Val32
- moved Ref4 160.7 mm to (134.2, -5.95), turned to 90 degrees
- moved Ref3 100.6 mm to (130.7, -5.95), turned to 90 degrees
- moved Ref9 92.5 mm to (-6.85, 69.9), turned to 180 degrees
- moved Ref7 83.0 mm to (130.7, 64.0), turned to 90 degrees
- moved Ref12 76.2 mm to (51.2, 73.5), turned to 180 degrees
- moved Ref10 71.5 mm to (-6.85, 73.5), turned to 180 degrees
- moved D15 69.5 mm to (117.9, 8.93)
- moved D2 55.7 mm to (0.00, 66.1), turned to 180 degrees
- moved D7 52.8 mm to (19.1, 8.93)
- moved D16 52.2 mm to (117.9, 47.0)
- moved D10 46.2 mm to (98.8, 66.1), turned to 180 degrees
- moved Ref11 38.9 mm to (51.2, 69.9), turned to 180 degrees
- moved D13 38.0 mm to (117.9, 28.0), turned to 180 degrees
- moved D3 38.0 mm to (0.00, 8.93), turned to 180 degrees
- moved D6 37.9 mm to (19.1, 66.1), turned to 180 degrees
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- renumbered D2 to D1, D20 to D10, D21 to D11, D23 to D12, D26 to D13, D28 to D14, D29 to D15, D31 to D16, D4 to D2, D5 to D3, D7 to D4, D10 to D5, D13 to D7, D15 to D8, D18 to D9, Ref8 to Rf8
Connections:
- D6 pad 1: Col1 -> Row3
- D6 pad 2: Row1 -> Net-(D6-Pad2)
- J1 pad A: Net-(J1-PadA) -> (no net)
- J2 pad A: Net-(J2-PadA) -> (no net)
- J3 pad A: Net-(J3-PadA) -> (no net)
- J4 pad A: Net-(J4-PadA) -> (no net)
- LED16 pad 1: Net-(LED16-Pad1) -> (no net)
- LED8 pad 1: Net-(LED8-Pad1) -> (no net)
- SW6 pad 2: Net-(D12-Pad2) (its old number) -> Net-(D6-Pad2)
- U1 pad 17: Net-(U1-Pad17) -> (no net)
- U1 pad 18: Net-(U1-Pad18) -> (no net)
- U1 pad 22: Net-(U1-Pad22) -> (no net)
- U1 pad 24: Net-(U1-Pad24) -> (no net)
- U1 pad 7: Net-(U1-Pad7) -> (no net)
- U2 pad 17: Net-(U2-Pad17) -> (no net)
- U2 pad 18: Net-(U2-Pad18) -> (no net)
- U2 pad 22: Net-(U2-Pad22) -> (no net)
- U2 pad 24: Net-(U2-Pad24) -> (no net)
- U2 pad 7: Net-(U2-Pad7) -> (no net)
Routing:
- net Net-(D15-Pad2): track 122.7 -> 6.80 mm, vias 1 -> 0
- net Net-(D2-Pad2): track 105.6 -> 6.96 mm, vias 1 -> 0
- net Net-(D16-Pad2): track 83.0 -> 6.80 mm, vias 1 -> 0
- net Net-(D13-Pad2): track 79.4 -> 6.93 mm, vias 1 -> 0
- net Net-(D7-Pad2): track 78.3 -> 6.88 mm
- net Col3r: track 164.5 -> 95.2 mm, vias 0 -> 2
- net Row0r: track 122.1 -> 71.7 mm, vias 0 -> 2
- net Net-(D1-Pad2): track 56.7 -> 6.89 mm, vias 2 -> 0
- net Net-(D4-Pad2): track 56.7 -> 6.96 mm
- net Net-(D3-Pad2): track 55.6 -> 6.96 mm, vias 2 -> 0
- net Col3: track 131.5 -> 83.2 mm, vias 2 -> 1
- net Col2: track 130.8 -> 84.6 mm, vias 0 -> 1
- net Row0: track 93.8 -> 49.3 mm
- net Row1r: track 109.5 -> 67.5 mm, vias 0 -> 2
- net Row2r: track 118.3 -> 77.9 mm, vias 0 -> 2
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
Commit message: add LOGO
Parts:
- added G***: LOGO, ロゴ:LTKeysLOGO, F.Cu at (71.4, 7.14)
- added G***: LOGO, ロゴ:LTKeysLOGO, F.Cu at (46.4, 6.55)
